File: kicad/fateful.kicad_sch (KiCad schematic)
At the start: 0 parts

Commit message: finished for today :D
Changed lines of the file:
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@@
 (kicad_sch
-	(version 20231120)
+	(version 20250114)
 	(generator "eeschema")
-	(generator_version "8.0")
+	(generator_version "9.0")
 	(paper "A4")
 	(sheet
-		(at 13.97 116.84)
-		(size 123.19 78.74)
+		(at 17.78 118.11)
+		(size 52.07 73.66)
+		(exclude_from_sim no)
+		(in_bom yes)
+		(on_board yes)
+		(dnp no)
 		(fields_autoplaced yes)
 		(stroke
@@
 		)
 		(property "Sheetname" "Control"
-			(at 13.97 116.1284 0)
+			(at 17.78 117.3984 0)
 			(effects
 				(font
@@
 		)
 		(property "Sheetfile" "control.kicad_sch"
-			(at 13.97 196.1646 0)
+			(at 17.78 192.3546 0)
 			(effects
 				(font
@@
 		)
 	)
+	(embedded_fonts no)
 )
