File: kicad/PC.kicad_sch (KiCad schematic)
At the start: 11 parts, among them U1 74LS161, U10 74HC04, U11 74HC04, U2 74LS161, U3 74LS161, U4 74LS161, U5 74HC04, U6 74HC04, U7 74LS08, U8 74HC04, U9 74HC04

Commit message: finished for today :D
Changed lines of the file:
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@@
 (kicad_sch
-	(version 20231120)
+	(version 20250114)
 	(generator "eeschema")
-	(generator_version "8.0")
+	(generator_version "9.0")
 	(paper "A4")
 	(junction

Commit message: changes i forgot to commit :sob:
Connections:
- net CLOCK renamed CLK
Other:
- moved on the sheet: U7D, U8A
Changed lines of the file:
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@@
 	(wire
 		(pts
-			(xy 25.4 138.43) (xy 25.4 149.86)
-		)
-		(stroke
-			(width 0)
-			(type default)
-		)
-	)
-	(wire
-		(pts
-			(xy 25.4 154.94) (xy 24.13 154.94)
+			(xy 25.4 138.43) (xy 25.4 151.13)
+		)
+		(stroke
+			(width 0)
+			(type default)
+		)
+	)
+	(wire
+		(pts
+			(xy 25.4 156.21) (xy 24.13 156.21)
 		)
 		(stroke
@@
 	(wire
 		(pts
-			(xy 21.59 119.38) (xy 24.13 119.38)
+			(xy 20.32 119.38) (xy 24.13 119.38)
 		)
 		(stroke
@@
 	(wire
 		(pts
-			(xy 24.13 154.94) (xy 24.13 119.38)
+			(xy 24.13 156.21) (xy 24.13 119.38)
 		)
 		(stroke
@@
 	(wire
 		(pts
+			(xy 120.65 153.67) (xy 120.65 152.4)
+		)
+		(stroke
+			(width 0)
+			(type default)
+		)
+	)
+	(wire
+		(pts
 			(xy 20.32 138.43) (xy 25.4 138.43)
 		)
@@
 	(wire
 		(pts
-			(xy 120.65 152.4) (xy 55.88 152.4)
+			(xy 120.65 153.67) (xy 55.88 153.67)
 		)
 		(stroke
@@
 			(width 0)
 			(type default)
-		)
-	)
-	(global_label "CLOCK"
-		(shape input)
-		(at 21.59 119.38 180)
-		(fields_autoplaced yes)
-		(effects
-			(font
-				(size 1.27 1.27)
-			)
-			(justify right)
-		)
-		(property "Intersheetrefs" "${INTERSHEET_REFS}"
-			(at 12.4362 119.38 0)
-			(effects
-				(font
-					(size 1.27 1.27)
-				)
-				(justify right)
-				(hide yes)
-			)
 		)
 	)
@@
 		(shape input)
 		(at 240.03 72.39 270)
+		(effects
+			(font
+				(size 1.27 1.27)
+			)
+			(justify right)
+		)
+	)
+	(hierarchical_label "CLK"
+		(shape input)
+		(at 20.32 119.38 180)
 		(effects
 			(font
@@
 	(symbol
 		(lib_id "74xx:74LS08")
-		(at 33.02 152.4 0)
+		(at 33.02 153.67 0)
 		(unit 4)
 		(exclude_from_sim no)
@@
 		(fields_autoplaced yes)
 		(property "Reference" "U7"
-			(at 33.0117 143.51 0)
+			(at 33.0117 144.78 0)
 			(effects
 				(font
@@
 		)
 		(property "Value" "74LS08"
-			(at 33.0117 146.05 0)
+			(at 33.0117 147.32 0)
 			(effects
 				(font
@@
 		)
 		(property "Footprint" ""
-			(at 33.02 152.4 0)
+			(at 33.02 153.67 0)
 			(effects
 				(font
@@
 		)
 		(property "Datasheet" "http://www.ti.com/lit/gpn/sn74LS08"
-			(at 33.02 152.4 0)
+			(at 33.02 153.67 0)
 			(effects
 				(font
@@
 		)
 		(property "Description" "Quad And2"
-			(at 33.02 152.4 0)
+			(at 33.02 153.67 0)
 			(effects
 				(font
@@
 	(symbol
 		(lib_id "74xx:74LS04")
-		(at 48.26 152.4 0)
+		(at 48.26 153.67 0)
 		(unit 1)
 		(exclude_from_sim no)
@@
 		(fields_autoplaced yes)
 		(property "Reference" "U8"
-			(at 48.26 143.51 0)
+			(at 48.26 144.78 0)
 			(effects
 				(font
@@
 		)
 		(property "Value" "74HC04"
-			(at 48.26 146.05 0)
+			(at 48.26 147.32 0)
 			(effects
 				(font
@@
 		)
 		(property "Footprint" ""
-			(at 48.26 152.4 0)
+			(at 48.26 153.67 0)
 			(effects
 				(font
@@
 		)
 		(property "Datasheet" "http://www.ti.com/lit/gpn/sn74LS04"
-			(at 48.26 152.4 0)
+			(at 48.26 153.67 0)
 			(effects
 				(font
@@
 		)
 		(property "Description" "Hex Inverter"
-			(at 48.26 152.4 0)
-			(effects
-				(font
+			(at 48.26 153.67 0)
+			(effects
+				(font
