File: kicad/control.kicad_sch (KiCad schematic)
At the start: 7 parts, among them U12 CAT28C16ALI90, U13 CAT28C16ALI90, U14 CAT28C16ALI90, U15 W27C512-45Z, U16 74HCT245, U17 74HCT245, U18 74LS04

Commit message: finished for today :D
Parts:
- added U19: 74HC377, symbol 74xx:74LS377
- added U20: 74HC161, symbol 74xx:74LS161
- added U21, U22, U23: 74HCT245, symbol 74xx:74LS245
- added U24: 74HC04, symbol 74xx:74LS04
- U15: value W27C512-45Z -> AT29C512-70PI; footprint 28P-DIP -> PDIP32_42P2X13P9_MCH; symbol W27C512:W27C512-45Z -> AT29C512:AT29C512-70PI
- U18: value 74LS04 -> 74HC04
Connections:
- net +5V: now also U15.31 (*WE), U15.32 (VCC), U19.20 (VCC), U20.9 (~{PE}), U22.1 (A->B), U22.20 (VCC), U23.1 (A->B), U23.20 (VCC)
- net GND: now also U15.16 (GND), U15.22 (*CE), U15.24 (*OE), U18.1, U19.10 (GND), U21.1 (A->B), U22.10 (GND), U23.10 (GND); no longer U18.2
- net ca.ca7: now reaches U13.1 (A7)
- net ca.ca7: now also U12.1 (A7)
- net ctrl.spd: now reaches U13.10 (I/O1)
- net ctrl.cr: now reaches U13.11 (I/O2)
- net ctrl.pci: now reaches U13.13 (I/O3)
- net ctrl.jnz: now reaches U13.14 (I/O4)
- net ctrl.li: now reaches U13.15 (I/O5)
- net ctrl.po: now reaches U13.16 (I/O6)
- net ctrl.sr: now reaches U13.17 (I/O7)
- net ca.ca6: now reaches U13.2 (A6)
- net ca.ca6: now also U12.2 (A6)
- net ca.ca5: now reaches U13.3 (A5)
- net ca.ca5: now also U12.3 (A5)
- net ca.ca4: now reaches U13.4 (A4)
- net ca.ca4: now also U12.4 (A4)
- net ca.ca3: now reaches U13.5 (A3)
- net ca.ca3: now also U12.5 (A3)
- net ca.ca2: now reaches U13.6 (A2)
- net ca.ca2: now also U12.6 (A2), U20.12 (Q2)
- net ca.ca1: now reaches U13.7 (A1)
- net ca.ca1: now also U12.7 (A1), U20.13 (Q1)
- net ca.ca0: now reaches U13.8 (A0)
- net ca.ca0: now also U12.8 (A0), U20.14 (Q0)
- net ctrl.spi: now reaches U13.9 (I/O0)
- net at U16.11 (B7): now also U15.27 (A8), U23.18 (B0); no longer U15.25 (A8)
- net at U16.12 (B6): now also U15.26 (A9), U23.17 (B1); no longer U15.24 (A9)
- net at U16.13 (B5): now also U15.23 (A10), U23.16 (B2); no longer U15.21 (A10)
- net at U16.14 (B4): now also U15.25 (A11), U23.15 (B3); no longer U15.23 (A11)
- net at U16.15 (B3): now also U15.4 (A12), U23.14 (B4); no longer U15.2 (A12)
- net at U16.16 (B2): now also U15.28 (A13), U23.13 (B5); no longer U15.26 (A13)
- net at U16.17 (B1): now also U15.29 (A14), U23.12 (B6); no longer U15.27 (A14)
- net at U16.18 (B0): now also U15.3 (A15), U23.11 (B7); no longer U15.1 (A15)
- net at U17.11 (B7): now also U15.12 (A0), U22.18 (B0); no longer U15.10 (A0)
- net at U17.12 (B6): now also U15.11 (A1), U22.17 (B1); no longer U15.9 (A1)
- net at U17.13 (B5): now also U15.10 (A2), U22.16 (B2); no longer U15.8 (A2)
- net at U17.14 (B4): now also U15.9 (A3), U22.15 (B3); no longer U15.7 (A3)
- net at U17.15 (B3): now also U15.8 (A4), U22.14 (B4); no longer U15.6 (A4)
- net at U17.16 (B2): now also U15.7 (A5), U22.13 (B5); no longer U15.5 (A5)
- net at U17.17 (B1): now also U15.6 (A6), U22.12 (B6); no longer U15.4 (A6)
- net at U17.18 (B0): now also U15.5 (A7), U22.11 (B7); no longer U15.3 (A7)
- net ctrl.aom: now reaches U12.10 (I/O1)
- net ctrl.aoh: now reaches U12.11 (I/O2)
- net ctrl.aoh: now also U12.9 (I/O0)
- net ctrl.ao: now reaches U12.13 (I/O3)
- net ctrl.rbi: now reaches U12.14 (I/O4)
- net ctrl.rbo: now reaches U12.15 (I/O5)
- net ctrl.rsb: now reaches U12.16 (I/O6)
- net ctrl.rsp: now reaches U12.17 (I/O7)
- net p.p0: now reaches U15.13 (I/O0)
- net p.p0: now also U19.3 (D0)
- net p.p1: now reaches U15.14 (I/O1)
- net p.p1: now also U19.4 (D1)
- net p.p2: now reaches U15.15 (I/O2)
- net p.p2: now also U19.7 (D2)
- net p.p3: now reaches U15.17 (I/O3)
- net p.p3: now also U19.8 (D3)
- net p.p4: now reaches U15.18 (I/O4)
- net p.p4: now also U19.13 (D4)
- net p.p5: now reaches U15.19 (I/O5)
- net p.p5: now also U19.14 (D5)
- net p.p6: now reaches U15.20 (I/O6)
- net p.p6: now also U19.17 (D6)
- new net: U18.2, U22.19 (CE), U23.19 (CE)
- new net: U20.2 (CP), U24.2
- new net: U20.10 (CET), U20.7 (CEP)
- new net CLOCK: U19.11 (CP), U24.1
- new net ah.ah0: U23.2 (A0)
- new net ah.ah1: U23.3 (A1)
- new net ah.ah2: U23.4 (A2)
- new net ah.ah3: U23.5 (A3)
- new net ah.ah4: U23.6 (A4)
- new net ah.ah5: U23.7 (A5)
- new net ah.ah6: U23.8 (A6)
- new net ah.ah7: U23.9 (A7)
- new net al.al0: U22.2 (A0)
- new net al.al1: U22.3 (A1)
- new net al.al2: U22.4 (A2)
- new net al.al3: U22.5 (A3)
- new net al.al4: U22.6 (A4)
- new net al.al5: U22.7 (A5)
- new net al.al6: U22.8 (A6)
- new net al.al7: U22.9 (A7)
- new net p.p7: U15.21 (I/O7), U19.18 (D7)
- no-connect marks 0 -> 6
Other:
- moved on the sheet: U14, U16, U17, U18A

Commit message: changes i forgot to commit :sob:
Parts:
- added U25, U33, U36: 74HC04, symbol 74xx:74LS04
- added U26, U31: 74LS32, symbol 74xx:74LS32
- added U27, U29, U30, U32: 74LS08, symbol 74xx:74LS08
- added U28: 74LS173, symbol 74xx:74LS173
- added U35: CD4044BE, CD4044BE:DIP794W45P254L1969H508Q16, symbol CD4044BE:CD4044BE
Connections:
- net +5V: now also U12.20 (*OE), U13.21 (*WE), U14.21 (*WE), U28.16 (VCC), U35.5 (EN), U35.8 (VSS)
- net CLOCK: now also U30.1
- net GND: now also U12.18 (*CE), U12.21 (*WE), U13.18 (*CE), U13.20 (*OE), U14.18 (*CE), U14.20 (*OE), U28.8 (GND), U35.16 (VDD)
- net Program Counter/JMP: now also U29.3
- net Program Counter/PCI: now also U31.3
- net ca.ca0: now also U14.8 (A0)
- net ca.ca1: now also U14.7 (A1)
- net ca.ca2: now also U14.6 (A2)
- net ca.ca3: now also U14.5 (A3), U19.9 (Q3)
- net ca.ca4: now also U14.4 (A4), U19.12 (Q4)
- net ca.ca5: now also U14.3 (A5), U19.15 (Q5)
- net ca.ca6: now also U14.2 (A6), U19.16 (Q6)
- net ca.ca7: now also U14.1 (A7), U19.19 (Q7)
- net ctrl.cr: now also U27.2, U28.11 (D3)
- net ctrl.li: now also U19.1 (~{E})
- net ctrl.la: now reaches U14.10 (I/O1)
- net ctrl.sa: now reaches U14.11 (I/O2)
- net ctrl.ali: now reaches U14.13 (I/O3)
- net ctrl.ahi: now reaches U14.14 (I/O4)
- net ctrl.lsp: now reaches U14.15 (I/O5)
- net ctrl.lpm: now reaches U14.16 (I/O6)
- net ctrl.sh: now reaches U14.17 (I/O7)
- net ctrl.thl: now reaches U14.9 (I/O0)
- net at U20.2 (CP), U24.2: now also U28.7 (Cp)
- net at U20.1 (~{MR}): now also U25.2
- net at U20.10 (CET), U20.7 (CEP): now also U30.2, U36.2
- new net: U31.1, U32.3
- new net: U26.1, U27.3
- new net: U25.1, U26.3
- new net: U27.1, U28.6 (Q3)
- new net: U29.1, U33.2
- new net: U35.13 (Q1), U36.1
- new net Program Counter/CLK: U30.3
- new net RESET: U26.2, U28.15 (Mr), U35.4 (R1)
Other:
- sheet Program Counter ports: added CLK; removed none
- moved on the sheet: U24A
